Commit message: fix: incorrect mesh directories

File: battle_bot_description/urdf/battle-bot.urdf (robot description, URDF)
Before this commit: robot battle-bot, 8 links, 7 joints
Links:
- link knee_mount: geometry collision mesh filename=package://battle_bot_description/meshes/knee_mount.stl; visual mesh filename=package://battle_bot_description/meshes/knee_mount.stl
- link left_foot: geometry collision mesh filename=package://battle_bot_description/meshes/left_foot.stl; visual mesh filename=package://battle_bot_description/meshes/left_foot.stl
- link part_1: geometry collision mesh filename=package://battle_bot_description/meshes/part_1.stl; visual mesh filename=package://battle_bot_description/meshes/part_1.stl
- link servo: geometry collision mesh filename=package://battle_bot_description/meshes/servo.stl; visual mesh filename=package://battle_bot_description/meshes/servo.stl
- link servo_2: geometry collision mesh filename=package://battle_bot_description/meshes/servo.stl; visual mesh filename=package://battle_bot_description/meshes/servo.stl
- link servo_3: geometry collision mesh filename=package://battle_bot_description/meshes/servo.stl; visual mesh filename=package://battle_bot_description/meshes/servo.stl
- link servo_4: geometry collision mesh filename=package://battle_bot_description/meshes/servo.stl; visual mesh filename=package://battle_bot_description/meshes/servo.stl
- link thigh_bracket: geometry collision mesh filename=package://battle_bot_description/meshes/thigh_bracket.stl; visual mesh filename=package://battle_bot_description/meshes/thigh_bracket.stl

Commit message: chore: change name of link in URDF

File: battle_bot_description/urdf/battle-bot.urdf (robot description, URDF)
Before this commit: robot battle-bot, 8 links, 7 joints
Links:
- removed link part_1
- added link ankle_mount, mass 0.00578055; collision mesh filename=package://battle_bot_description/meshes/ankle_mount.stl; visual mesh filename=package://battle_bot_description/meshes/ankle_mount.stl
Joints:
- joint ankle: parent part_1 -> ankle_mount
- joint ankle_servo_v: child part_1 -> ankle_mount
