Commit message: chore: use xacro

File: battle_bot_description/urdf/battle-bot.urdf.xacro (robot description, xacro)
@@ -1,3 +1,4 @@
-<robot name="battle-bot">
+<?xml version="1.0"?>
+<robot xmlns:xacro="http://www.ros.org/wiki/xacro" name="battle-bot">
 <link name="thigh_bracket">
 <visual>
@@ -200,5 +201,5 @@
 </inertial>
 </link>
-<joint name="ankle_servo_h" type="revolute">
+<joint name="ankle_servo_h" type="continuous">
 <origin xyz="0.00575 0.0237939 -0.00575" rpy="-1.5708 -1.5708 0" />
 <parent link="servo_4" />
@@ -216,5 +217,5 @@
 <joint_properties friction="0.0"/>
 </joint>
-<joint name="ankle_servo_v" type="revolute">
+<joint name="ankle_servo_v" type="continuous">
 <origin xyz="0.0195 6.93889e-18 0.017" rpy="5.52479e-16 -4.02837e-16 1.17242" />
 <parent link="servo_3" />
@@ -232,5 +233,5 @@
 <joint_properties friction="0.0"/>
 </joint>
-<joint name="knee_servo" type="revolute">
+<joint name="knee_servo" type="continuous">
 <origin xyz="0 -0.023 -0.01725" rpy="-1.5708 0.474293 -3.18767e-16" />
 <parent link="servo_2" />
@@ -248,5 +249,5 @@
 <joint_properties friction="0.0"/>
 </joint>
-<joint name="thigh_servo" type="revolute">
+<joint name="thigh_servo" type="continuous">
 <origin xyz="0.0813147 0.0614459 -0.0195855" rpy="1.5708 -0.959931 -3.87553e-14" />
 <parent link="thigh_bracket" />
@@ -256,3 +257,39 @@
 <joint_properties friction="0.0"/>
 </joint>
+<transmission name="ankle_servo_v_trans">
+  <type>transmission_interface/SimpleTransmission</type>
+  <actuator name="$ankle_servo_v_motor">
+    <mechanicalReduction>1</mechanicalReduction>
+  </actuator>
+  <joint name="ankle_servo_v">
+    <hardwareInterface>hardware_interface/PositionJointInterface</hardwareInterface>
+  </joint>
+</transmission>
+<transmission name="ankle_servo_v_trans">
+  <type>transmission_interface/SimpleTransmission</type>
+  <actuator name="$ankle_servo_v_motor">
+    <mechanicalReduction>1</mechanicalReduction>
+  </actuator>
+  <joint name="ankle_servo_v">
+    <hardwareInterface>hardware_interface/PositionJointInterface</hardwareInterface>
+  </joint>
+</transmission>
+<transmission name="knee_servo_trans">
+  <type>transmission_interface/SimpleTransmission</type>
+  <actuator name="$knee_servo_motor">
+    <mechanicalReduction>1</mechanicalReduction>
+  </actuator>
+  <joint name="knee_servo">
+    <hardwareInterface>hardware_interface/PositionJointInterface</hardwareInterface>
+  </joint>
+</transmission>
+<transmission name="thigh_servo_trans">
+  <type>transmission_interface/SimpleTransmission</type>
+  <actuator name="$thigh_servo_motor">
+    <mechanicalReduction>1</mechanicalReduction>
+  </actuator>
+  <joint name="thigh_servo">
+    <hardwareInterface>hardware_interface/PositionJointInterface</hardwareInterface>
+  </joint>
+</transmission>
 </robot>
